File: matrix.kicad_sch (KiCad schematic)
At the start: 202 parts, among them SW1 ?, SW10 ?, SW100 ?, SW101 ?, SW102 ?, SW103 ?, SW104 ?, SW11 ?, SW12 ?, SW13 ?, SW14 ?, SW15 ?, SW16 ?, SW17 ?, SW18 ?, SW19 ?, SW2 ?, SW20 ?, SW21 ?, SW22 ?, SW23 ?, SW24 ?, SW25 ?, SW26 ?, SW27 ?, SW28 ?, SW29 ?, SW3 ?, SW30 ?, SW31 ?, SW32 ?, SW33 ?, SW34 ?, SW35 ?, SW36 ?, SW37 ?, SW38 ?, SW39 ?, SW4 ?, SW40 ?, SW41 ?, SW42 ?, SW43 ?, SW44 ?, SW45 ?, SW46 ?, SW47 ?, SW48 ?, SW49 ?, SW5 ?, SW50 ?, SW51 ?, SW52 ?, SW53 ?, SW54 ?, SW55 ?, SW56 ?, SW57 ?, SW58 ?, SW59 ?, SW6 ?, SW60 ?, SW61 ?, SW62 ?, SW63 ?, SW64 ?, SW65 ?, SW66 ?, SW67 ?, SW68 ?, SW69 ?, SW7 ?, SW70 ?, SW71 ?, SW72 ?, SW73 ?, SW74 ?, SW75 ?, SW76 ?, SW77 ?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

Commit message: Initial Commit
Parts:
- removed D90, D91: D, Diode_SMD:D_SOD-123, symbol Device:D_Small
- removed S7: 7U_SPACE, marbastlib-mx:STAB_MX_7u, symbol marbastlib-mx:MX_stab
- removed SW1, SW102, SW103, SW104, SW13, SW14, SW15, SW16, SW17, SW18, SW19, SW20, SW21, SW22, SW23, SW24, SW25, SW26, SW27, SW28, SW29, SW30, SW31, SW32, SW33, SW34, SW35, SW36, SW38, SW39, SW40, SW41, SW42, SW43, SW44, SW45, SW46, SW47, SW48, SW49, SW51, SW52, SW53, SW54, SW57, SW58, SW59, SW60, SW61, SW62, SW63, SW64, SW65, SW66, SW67, SW68, SW69, SW71, SW72, SW73, SW74, SW75, SW76, SW77, SW78, SW79, SW80, SW81, SW82, SW84, SW85, SW86, SW90, SW93, SW94, SW98: ?, marbastlib-mx:SW_MX_HS_1u, symbol marbastlib-mx:MX_SW_HS
- removed SW100, SW37, SW50, SW88, SW92, SW96: ?, marbastlib-mx:SW_MX_HS_1.5u, symbol marbastlib-mx:MX_SW_HS
- removed SW101, SW70, SW87, SW89, SW91, SW95, SW97, SW99: ?, marbastlib-mx:SW_MX_HS_1.25u, symbol marbastlib-mx:MX_SW_HS
- removed SW55: ?, marbastlib-mx:SW_MX_HS_1.75u_stp, symbol marbastlib-mx:MX_SW_HS
- removed SW56, SW83: ?, marbastlib-mx:SW_MX_HS_1.75u, symbol marbastlib-mx:MX_SW_HS
- added SW"1, SW#1, SW-1, SW;1, SW<1, SW=1, SW>1, SWESC1, SWF1, SW[1, SW\2, SW]1, SWa1, SWalt1, SWalt2, SWansient1, SWb1, SWbs1, SWbs2, SWc1, SWcaps1, SWcd1, SWcd2, SWctrl1, SWctrl2, SWd1, SWdel1, SWdown1, SWe1, SWend1, SWf10, SWf11, SWf12, SWf13, SWf14, SWf2, SWf3, SWf4, SWf5, SWf6, SWf7, SWf8, SWf9, SWg1, SWh1, SWhome1, SWi1, SWinsert1, SWisoenter1, SWj1, SWk1, SWl1, SWleft1, SWlshift1, SWm1, SWmisc1, SWn1, SWo1, SWp1, SWpausebreak1, SWpgdn1, SWpgup1, SWprtsc1, SWq1, SWr1, SWright1, SWrshift1, SWs1, SWsclock1, SWspace1, SWt1, SWtab1, SWu1, SWup1, SWv1, SWw1, SWx1, SWy1, SWz1, SW|\1, SW~1: MX_SW_HS, marbastlib-mx:SW_MX_HS_1u, symbol marbastlib-mx:MX_SW_HS
- added SWshift1, SWstcaps2: (no value), marbastlib-mx:SW_MX_HS_1u, symbol marbastlib-mx:MX_SW_HS
- D1, D10, D11, D12, D13, D14, D15, D16, D17, D18, D19, D2, D20, D21, D22, D23, D24, D25, D26, D27, D28, D29, D3, D30, D31, D32, D33, D34, D35, D36, D37, D38, D39, D4, D40, D41, D42, D43, D44, D45, D46, D47, D48, D49, D5, D50, D51, D52, D53, D54, D55, D56, D57, D58, D59, D6, D60, D61, D62, D63, D64, D65, D66, D67, D68, D69, D7, D70, D71, D72, D73, D74, D75, D76, D77, D78, D79, D8, D80, D81, D82, D83, D84, D85, D86, D87, D88, D89, D9: value D -> D_Small
- S1: value BACKSPACE -> LSHIFT; footprint marbastlib-mx:STAB_MX_2u -> marbastlib-mx:STAB_MX_2.25u
- S2: value ISO_ENTER -> 7U_SPACE; footprint marbastlib-mx:STAB_MX_ISO_FLIPPED -> marbastlib-mx:STAB_MX_7u
- S3: value ANSI_ENTER -> ISO_ENTER; footprint marbastlib-mx:STAB_MX_2.25u -> marbastlib-mx:STAB_MX_ISO_FLIPPED
- S4: value LSHIFT -> RSHIFT; footprint marbastlib-mx:STAB_MX_2.25u -> marbastlib-mx:STAB_MX_2.75u
- S5: value RSHIFT -> ANSI_ENTER; footprint marbastlib-mx:STAB_MX_2.75u -> marbastlib-mx:STAB_MX_2.25u
- S6: value 6.25U_SPACE -> BACKSPACE; footprint marbastlib-mx:STAB_MX_6.25u -> marbastlib-mx:STAB_MX_2u
- SW10, SW11, SW12, SW2, SW3, SW4, SW5, SW6, SW7, SW8, SW9: value ? -> MX_SW_HS
Connections:
- net COL0: now also SWESC1.1, SWcaps1.2, SWctrl1.1, SWlshift1.2, SWshift1.1, SWstcaps2.1, SWtab1.1, SW~1.1
- net COL1: now also SWF1.1, SWa1.1, SWcd1.1, SWq1.1, SW|\1.1
- net COL10: now also SW;1.1, SW>1.1, SWalt2.1, SWf11.1, SWp1.1
- net COL11: now also SW"1.1, SW-1.1, SW[1.1, SWf12.1
- net COL12: now also SW#1.2, SW=1.1, SW]1.1, SWansient1.1, SWcd2.1, SWf13.1, SWrshift1.1
- net COL13: now also SW\2.2, SWbs1.1, SWbs2.1, SWf14.1, SWisoenter1.1, SWmisc1.2
- net COL14: now also SWdel1.1, SWinsert1.1, SWleft1.1, SWprtsc1.1
- net COL15: now also SWdown1.1, SWend1.1, SWhome1.1, SWsclock1.1, SWup1.1
- net COL16: now also SWpausebreak1.1, SWpgdn1.1, SWpgup1.1, SWright1.1
- net COL2: now also SWalt1.1, SWf2.1, SWs1.1, SWw1.1, SWz1.1
- net COL3: now also SWd1.1, SWe1.1, SWf3.1, SWx1.1
- net COL4: now also SWc1.1, SWf4.1, SWf5.1, SWr1.1
- net COL5: now also SWf6.1, SWg1.1, SWt1.1, SWv1.1
- net COL6: now also SWb1.1, SWf7.1, SWh1.1, SWspace1.1, SWy1.1
- net COL7: now also SWf8.1, SWj1.1, SWn1.1, SWu1.1
- net COL8: now also SWf9.1, SWi1.1, SWk1.1, SWm1.1
- net COL9: now also SW<1.1, SWf10.1, SWl1.1, SWo1.1
- net ROW0: now also D19.1 (K), D24.1 (K), D29.1 (K), D34.1 (K), D40.1 (K), D45.1 (K), D50.1 (K), D55.1 (K), D61.1 (K), D66.1 (K), D74.1 (K), D77.1 (K), D81.1 (K), D86.1 (K); no longer D10.1 (K), D11.1 (K), D12.1 (K), D14.1 (K), D15.1 (K), D16.1 (K), D17.1 (K), D2.1 (K), D3.1 (K), D4.1 (K), D5.1 (K), D6.1 (K), D8.1 (K), D9.1 (K)
- net ROW1: now also D14.1 (K), D2.1 (K), D41.1 (K), D46.1 (K), D51.1 (K), D56.1 (K), D62.1 (K), D67.1 (K), D73.1 (K), D75.1 (K), D78.1 (K), D8.1 (K), D82.1 (K), D87.1 (K); no longer D18.1 (K), D19.1 (K), D21.1 (K), D22.1 (K), D23.1 (K), D24.1 (K), D26.1 (K), D27.1 (K), D28.1 (K), D29.1 (K), D31.1 (K), D33.1 (K), D34.1 (K)
- net ROW2: now also D15.1 (K), D21.1 (K), D26.1 (K), D3.1 (K), D31.1 (K), D57.1 (K), D63.1 (K), D68.1 (K), D76.1 (K), D79.1 (K), D83.1 (K), D88.1 (K), D9.1 (K); no longer D37.1 (K), D38.1 (K), D39.1 (K), D40.1 (K), D41.1 (K), D43.1 (K), D44.1 (K), D45.1 (K), D46.1 (K), D48.1 (K), D49.1 (K), D50.1 (K), D51.1 (K)
- net ROW3: now also D10.1 (K), D16.1 (K), D22.1 (K), D27.1 (K), D37.1 (K), D4.1 (K), D43.1 (K), D48.1 (K), D69.1 (K); no longer D54.1 (K), D55.1 (K), D56.1 (K), D57.1 (K), D59.1 (K), D60.1 (K), D61.1 (K), D62.1 (K), D63.1 (K), D65.1 (K)
- net ROW4: now also D11.1 (K), D17.1 (K), D23.1 (K), D28.1 (K), D33.1 (K), D38.1 (K), D44.1 (K), D49.1 (K), D5.1 (K), D54.1 (K), D59.1 (K), D65.1 (K), D84.1 (K); no longer D66.1 (K), D67.1 (K), D68.1 (K), D69.1 (K), D71.1 (K), D72.1 (K), D73.1 (K), D74.1 (K), D75.1 (K), D76.1 (K), D77.1 (K), D78.1 (K), D79.1 (K), D80.1 (K)
- net ROW5: now also D12.1 (K), D18.1 (K), D39.1 (K), D6.1 (K), D60.1 (K), D71.1 (K), D72.1 (K), D80.1 (K); no longer D81.1 (K), D82.1 (K), D83.1 (K), D84.1 (K), D86.1 (K), D87.1 (K), D88.1 (K)
- net at D15.2 (A): now also SWw1.2
- net at D21.2 (A): now also SWe1.2
- net at D64.2 (A): now also SW"1.2
- net at D66.2 (A): now also SWf13.2
- net at D46.2 (A): now also SW9.2
- net at D41.2 (A): now also SW8.2
- net at D56.2 (A): now also SW11.2
- net at D6.2 (A): now also SWctrl1.2; no longer SW6.2
- net at D67.2 (A): now also SW=1.2
- net at D78.2 (A): now also SWinsert1.2
- net at D16.2 (A): now also SWs1.2
- net at D18.2 (A): now also SWalt1.2
- net at D89.2 (A): now also SWright1.2
- net at D24.2 (A): now also SWf4.2
- net at D84.2 (A): now also SWup1.2
- net at D31.2 (A): now also SWt1.2
- net at D62.2 (A): now also SW-1.2
- net at D83.2 (A): now also SWend1.2
- net at D7.2 (A): now also SWF1.2; no longer SW7.2
- net at SW12.2: now also D65.2 (A); no longer D12.2 (A)
- net at D35.2 (A): now also SW7.2
- net at D58.2 (A): now also SW;1.2
- net at D70.2 (A): now also SWrshift1.2
- net at D14.2 (A): now also SW3.2
- net at D49.2 (A): now also SWm1.2
- net at D71.2 (A): now also SWcd2.2
- net at D8.2 (A): now also SW2.2; no longer SW8.2
- net at D50.2 (A): now also SWf10.2
- net at D52.2 (A): now also SWo1.2
- net at D74.2 (A): now also SWf14.2
- net at D28.2 (A): now also SWc1.2
- net at D88.2 (A): now also SWpgdn1.2
- net at D27.2 (A): now also SWf5.2
- net at D79.2 (A): now also SWdel1.2
- net at D77.2 (A): now also SWprtsc1.2
- net at D37.2 (A): now also SWh1.2
- net at D75.2 (A): now also SWmisc1.1
- net at D34.2 (A): now also SWf7.2
- net at D9.2 (A): now also SWq1.2; no longer SW9.2
- net at SW4.2: now also D20.2 (A); no longer D4.2 (A)
- net at D47.2 (A): now also SWi1.2
- net at D85.2 (A): now also SWdown1.2
- net at D10.2 (A): now also SWa1.2; no longer SW10.2
- net at D42.2 (A): now also SWu1.2
- net at D54.2 (A): now also SW<1.2
- net at D38.2 (A): now also SWb1.2
- net at D33.2 (A): now also SWv1.2
- net at D73.2 (A): now also SWbs1.2, SWbs2.2
- net at D76.2 (A): now also SW\2.1, SWisoenter1.2
- net at D86.2 (A): now also SWpausebreak1.2
- net at D87.2 (A): now also SWpgup1.2
- net at D29.2 (A): now also SWf6.2
- net at D30.2 (A): now also SW6.2
- net at D44.2 (A): now also SWn1.2
- net at D72.2 (A): now also SWctrl2.2
- net at D13.2 (A): now also SWf2.2
- net at D80.2 (A): now also SWleft1.2
- net at D19.2 (A): now also SWf3.2
- net at D82.2 (A): now also SWhome1.2
- net at D59.2 (A): now also SW>1.2
- net at D23.2 (A): now also SWx1.2
- net at D39.2 (A): now also SWspace1.2
- net at D40.2 (A): now also SWf8.2
- net at D51.2 (A): now also SW10.2
- net at D45.2 (A): now also SWf9.2
- net at D36.2 (A): now also SWy1.2
- net at D61.2 (A): now also SWf12.2
- net at D25.2 (A): now also SW5.2
- net at D22.2 (A): now also SWd1.2
- net at D43.2 (A): now also SWj1.2
- net at D48.2 (A): now also SWk1.2
- net at D2.2 (A): now also SW~1.2; no longer SW2.2
- net at D17.2 (A): now also SWz1.2
- net at D11.2 (A): now also SW|\1.2; no longer SW11.2
- net at D26.2 (A): now also SWr1.2
- net at D57.2 (A): now also SWp1.2
- net at D60.2 (A): now also SWalt2.2
- net at D5.2 (A): now also SWlshift1.1, SWshift1.2; no longer SW5.2
- net at D3.2 (A): now also SWtab1.2; no longer SW3.2
- net at D69.2 (A): now also SW#1.1, SWansient1.2
- net at D81.2 (A): now also SWsclock1.2
- net at D68.2 (A): now also SW]1.2
- net at D32.2 (A): now also SWg1.2
- net at D1.2 (A): now also SWESC1.2
- net at D53.2 (A): now also SWl1.2
- net at D55.2 (A): now also SWf11.2
- net at D63.2 (A): now also SW[1.2
- new net: D4.2 (A), SWcaps1.1, SWstcaps2.2
- new net: D12.2 (A), SWcd1.2
Other:
- company: (none) -> Nullus Studios
- title: (none) -> nullus v1 PCB (UDB COMPATIBLE)
